File: kicad_6_docs/CV_generators.kicad_sch (KiCad schematic)
At the start: 21 parts, among them J4 1/4"_jack, U12 TL072, U13 TL072

Commit message: Fix power supply errors, tidy up schematic
Changed lines of the file:
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@@
   (title_block
     (title "A.P. Joystick VCF pedal")
-    (date "2022-01-14")
+    (date "2022-08-01")
     (rev "0")
     (comment 2 "creativecommons.org/licenses/by/4.0")
@@
       (effects (font (size 1.27 1.27)) hide)
     )
+    (pin "1")
+    (pin "2")
+    (pin "3")
     (pin "5")
     (pin "6")
     (pin "7")
+    (pin "4")
+    (pin "8")
   )
   (symbol (lib_id "Amplifier_Operational:TL072") (at 229.87 140.97 0) (mirror x) (unit 2)
@@
       (effects (font (size 1.27 1.27)) hide)
     )
+    (pin "1")
+    (pin "2")
+    (pin "3")
     (pin "5")
     (pin "6")
     (pin "7")
+    (pin "4")
+    (pin "8")
   )
   (symbol (lib_id "Diode:1N4148") (at 204.47 144.78 90) (unit 1)
@@
     (pin "2")
     (pin "3")
+    (pin "5")
+    (pin "6")
+    (pin "7")
+    (pin "4")
+    (pin "8")
   )
   (symbol (lib_id "power:GND") (at 133.35 33.02 0) (unit 1)
@@
     (fill (color 0 0 0 0.0000))
     (property "Sheet name" "LFO" (id 0) (at 50.8 34.8484 0)
-      (effects (font (size 1.27 1.27)) (justify left bottom))
+      (effects (font (size 1.7 1.7)) (justify left bottom))
     )
     (property "Sheet file" "LFO.kicad_sch" (id 1) (at 50.8 74.2446 0)
-      (effects (font (size 1.27 1.27)) (justify left top))
+      (effects (font (size 1.27 1.27)) (justify left top) hide)
     )
     (pin "LFO_OUT" output (at 76.2 40.64 0)
@@
     (fill (color 0 0 0 0.0000))
     (property "Sheet name" "joystick" (id 0) (at 50.8 130.0984 0)
-      (effects (font (size 1.27 1.27)) (justify left bottom))
+      (effects (font (size 1.7 1.7)) (justify left bottom))
     )
     (property "Sheet file" "joystick.kicad_sch" (id 1) (at 50.8 169.4946 0)
-      (effects (font (size 1.27 1.27)) (justify left top))
+      (effects (font (size 1.27 1.27)) (justify left top) hide)
     )
     (pin "X_OUT" output (at 76.2 138.43 0)
@@
     (fill (color 0 0 0 0.0000))
     (property "Sheet name" "envelope_follower" (id 0) (at 50.8 83.1084 0)
-      (effects (font (size 1.27 1.27)) (justify left bottom))
+      (effects (font (size 1.7 1.7)) (justify left bottom))
     )
     (property "Sheet file" "envelope_follower.kicad_sch" (id 1) (at 50.8 122.5046 0)
-      (effects (font (size 1.27 1.27)) (justify left top))
+      (effects (font (size 1.27 1.27)) (justify left top) hide)
     )
     (pin "ENVELOPE_OUT" output (at 76.2 86.36 0)
